File: elec/layout/default/analog-keyboard-handwiring-module.kicad_pcb (KiCad board)
At the start: 2 copper layers, 225.7 x 100.8 mm, 0 parts

Commit message: Add pre-ato version of the board
Parts:
- added C1: 0.1µF, Capacitor_SMD:C_0805_2012Metric_Pad1.18x1.45mm_HandSolder, F.Cu at (114.4, 64.1)
- added C10: 0.1µF, Capacitor_SMD:C_0805_2012Metric_Pad1.18x1.45mm_HandSolder, F.Cu at (95.6, 55.3)
- added C11: 0.1µF, Capacitor_SMD:C_0805_2012Metric_Pad1.18x1.45mm_HandSolder, F.Cu at (114.4, 83.1)
- added C12: 0.1µF, Capacitor_SMD:C_0805_2012Metric_Pad1.18x1.45mm_HandSolder, F.Cu at (114.7, 74.3)
- added C13: 0.1µF, Capacitor_SMD:C_0805_2012Metric_Pad1.18x1.45mm_HandSolder, F.Cu at (76.3, 83.1)
- added C14: 0.1µF, Capacitor_SMD:C_0805_2012Metric_Pad1.18x1.45mm_HandSolder, F.Cu at (76.6, 74.3)
- added C15: 0.1µF, Capacitor_SMD:C_0805_2012Metric_Pad1.18x1.45mm_HandSolder, F.Cu at (133.4, 83.1)
- added C16: 0.1µF, Capacitor_SMD:C_0805_2012Metric_Pad1.18x1.45mm_HandSolder, F.Cu at (133.7, 74.3)
- added C17: 0.1µF, Capacitor_SMD:C_0805_2012Metric_Pad1.18x1.45mm_HandSolder, F.Cu at (57.2, 83.1)
- added C18: 0.1µF, Capacitor_SMD:C_0805_2012Metric_Pad1.18x1.45mm_HandSolder, F.Cu at (57.5, 74.3)
- added C19: 0.1µF, Capacitor_SMD:C_0805_2012Metric_Pad1.18x1.45mm_HandSolder, F.Cu at (95.3, 83.1)
- added C2: 0.1µF, Capacitor_SMD:C_0805_2012Metric_Pad1.18x1.45mm_HandSolder, F.Cu at (114.7, 55.3)
- added C20: 0.1µF, Capacitor_SMD:C_0805_2012Metric_Pad1.18x1.45mm_HandSolder, F.Cu at (95.6, 74.3)
- added C21: 0.1µF, Capacitor_SMD:C_0805_2012Metric_Pad1.18x1.45mm_HandSolder, F.Cu at (133.4, 102.2)
- added C22: 0.1µF, Capacitor_SMD:C_0805_2012Metric_Pad1.18x1.45mm_HandSolder, F.Cu at (133.7, 93.4)
- added C23: 0.1µF, Capacitor_SMD:C_0805_2012Metric_Pad1.18x1.45mm_HandSolder, F.Cu at (95.3, 102.2)
- added C24: 0.1µF, Capacitor_SMD:C_0805_2012Metric_Pad1.18x1.45mm_HandSolder, F.Cu at (95.6, 93.4)
- added C25: 0.1µF, Capacitor_SMD:C_0805_2012Metric_Pad1.18x1.45mm_HandSolder, F.Cu at (76.3, 102.2)
- added C26: 0.1µF, Capacitor_SMD:C_0805_2012Metric_Pad1.18x1.45mm_HandSolder, F.Cu at (76.6, 93.4)
- added C27: 0.1µF, Capacitor_SMD:C_0805_2012Metric_Pad1.18x1.45mm_HandSolder, F.Cu at (57.2, 102.2)
- added C28: 0.1µF, Capacitor_SMD:C_0805_2012Metric_Pad1.18x1.45mm_HandSolder, F.Cu at (57.5, 93.4)
- added C29: 0.1µF, Capacitor_SMD:C_0805_2012Metric_Pad1.18x1.45mm_HandSolder, F.Cu at (114.4, 102.2)
- added C3: 0.1µF, Capacitor_SMD:C_0805_2012Metric_Pad1.18x1.45mm_HandSolder, F.Cu at (133.4, 64.1)
- added C30: 0.1µF, Capacitor_SMD:C_0805_2012Metric_Pad1.18x1.45mm_HandSolder, F.Cu at (114.7, 93.4)
- added C31: 0.1µF, Capacitor_SMD:C_0805_2012Metric_Pad1.18x1.45mm_HandSolder, F.Cu at (133.4, 121.2)
- added C32: 0.1µF, Capacitor_SMD:C_0805_2012Metric_Pad1.18x1.45mm_HandSolder, F.Cu at (133.7, 112.4)
- added C33: 0.1µF, Capacitor_SMD:C_0805_2012Metric_Pad1.18x1.45mm_HandSolder, F.Cu at (95.3, 121.2)
- added C34: 0.1µF, Capacitor_SMD:C_0805_2012Metric_Pad1.18x1.45mm_HandSolder, F.Cu at (95.6, 112.4)
- added C35: 0.1µF, Capacitor_SMD:C_0805_2012Metric_Pad1.18x1.45mm_HandSolder, F.Cu at (114.4, 121.2)
- added C36: 0.1µF, Capacitor_SMD:C_0805_2012Metric_Pad1.18x1.45mm_HandSolder, F.Cu at (114.7, 112.4)
- added C37: 0.1µF, Capacitor_SMD:C_0805_2012Metric_Pad1.18x1.45mm_HandSolder, F.Cu at (57.2, 121.2)
- added C38: 0.1µF, Capacitor_SMD:C_0805_2012Metric_Pad1.18x1.45mm_HandSolder, F.Cu at (57.5, 112.4)
- added C39: 0.1µF, Capacitor_SMD:C_0805_2012Metric_Pad1.18x1.45mm_HandSolder, F.Cu at (76.3, 121.2)
- added C4: 0.1µF, Capacitor_SMD:C_0805_2012Metric_Pad1.18x1.45mm_HandSolder, F.Cu at (133.7, 55.3)
- added C40: 0.1µF, Capacitor_SMD:C_0805_2012Metric_Pad1.18x1.45mm_HandSolder, F.Cu at (76.6, 112.4)
- added C41: 0.1µF, Capacitor_SMD:C_0805_2012Metric_Pad1.18x1.45mm_HandSolder, F.Cu at (57.2, 140.3)
- added C42: 0.1µF, Capacitor_SMD:C_0805_2012Metric_Pad1.18x1.45mm_HandSolder, F.Cu at (57.5, 131.5)
- added C43: 0.1µF, Capacitor_SMD:C_0805_2012Metric_Pad1.18x1.45mm_HandSolder, F.Cu at (95.3, 140.3)
- added C44: 0.1µF, Capacitor_SMD:C_0805_2012Metric_Pad1.18x1.45mm_HandSolder, F.Cu at (95.6, 131.5)
- added C45: 0.1µF, Capacitor_SMD:C_0805_2012Metric_Pad1.18x1.45mm_HandSolder, F.Cu at (114.4, 140.3)
- added C46: 0.1µF, Capacitor_SMD:C_0805_2012Metric_Pad1.18x1.45mm_HandSolder, F.Cu at (114.7, 131.5)
- added C47: 0.1µF, Capacitor_SMD:C_0805_2012Metric_Pad1.18x1.45mm_HandSolder, F.Cu at (133.4, 140.3)
- added C48: 0.1µF, Capacitor_SMD:C_0805_2012Metric_Pad1.18x1.45mm_HandSolder, F.Cu at (133.7, 131.5)
- added C49: 0.1µF, Capacitor_SMD:C_0805_2012Metric_Pad1.18x1.45mm_HandSolder, F.Cu at (76.3, 140.3)
- added C5: 0.1µF, Capacitor_SMD:C_0805_2012Metric_Pad1.18x1.45mm_HandSolder, F.Cu at (57.2, 64.1)
- added C50: 0.1µF, Capacitor_SMD:C_0805_2012Metric_Pad1.18x1.45mm_HandSolder, F.Cu at (76.6, 131.5)
- added C6: 0.1µF, Capacitor_SMD:C_0805_2012Metric_Pad1.18x1.45mm_HandSolder, F.Cu at (57.5, 55.3)
- added C7: 0.1µF, Capacitor_SMD:C_0805_2012Metric_Pad1.18x1.45mm_HandSolder, F.Cu at (76.3, 64.1)
- added C8: 0.1µF, Capacitor_SMD:C_0805_2012Metric_Pad1.18x1.45mm_HandSolder, F.Cu at (76.6, 55.3)
- added C9: 0.1µF, Capacitor_SMD:C_0805_2012Metric_Pad1.18x1.45mm_HandSolder, F.Cu at (95.3, 64.1)
- added H1: MountingHole, MountingHole:MountingHole_2.2mm_M2, F.Cu at (69.0, 59.5)
- added H10: MountingHole, MountingHole:MountingHole_2.2mm_M2, F.Cu at (69.0, 78.6)
- added H11: MountingHole, MountingHole:MountingHole_2.2mm_M2, F.Cu at (88.1, 78.6)
- added H13: MountingHole, MountingHole:MountingHole_2.2mm_M2, F.Cu at (126.2, 78.6)
- added H14: MountingHole, MountingHole:MountingHole_2.2mm_M2, F.Cu at (59.5, 88.1)
- added H15: MountingHole, MountingHole:MountingHole_2.2mm_M2, F.Cu at (78.6, 88.1)
- added H16: MountingHole, MountingHole:MountingHole_2.2mm_M2, F.Cu at (97.6, 88.1)
- added H17: MountingHole, MountingHole:MountingHole_2.2mm_M2, F.Cu at (116.7, 88.1)
- added H18: locked, MountingHole:MountingHole_2.2mm_M2, F.Cu at (135.7, 88.1)
- added H19: MountingHole, MountingHole:MountingHole_2.2mm_M2, F.Cu at (69.0, 97.6)
- added H2: MountingHole, MountingHole:MountingHole_2.2mm_M2, F.Cu at (88.1, 59.5)
- added H20: MountingHole, MountingHole:MountingHole_2.2mm_M2, F.Cu at (88.1, 97.6)
- added H21: MountingHole, MountingHole:MountingHole_2.2mm_M2, F.Cu at (107.2, 97.6)
- added H22: MountingHole, MountingHole:MountingHole_2.2mm_M2, F.Cu at (126.2, 97.6)
- added H23: MountingHole, MountingHole:MountingHole_2.2mm_M2, F.Cu at (59.5, 107.2)
- added H24: MountingHole, MountingHole:MountingHole_2.2mm_M2, F.Cu at (78.6, 107.2)
- added H25: MountingHole, MountingHole:MountingHole_2.2mm_M2, F.Cu at (97.6, 107.2)
- added H26: MountingHole, MountingHole:MountingHole_2.2mm_M2, F.Cu at (116.7, 107.2)
- added H27: MountingHole, MountingHole:MountingHole_2.2mm_M2, F.Cu at (135.7, 107.2)
- added H28: MountingHole, MountingHole:MountingHole_2.2mm_M2, F.Cu at (69.0, 116.7)
- added H29: MountingHole, MountingHole:MountingHole_2.2mm_M2, F.Cu at (88.1, 116.7)
- added H3: MountingHole, MountingHole:MountingHole_2.2mm_M2, F.Cu at (107.2, 59.5)
- added H30: MountingHole, MountingHole:MountingHole_2.2mm_M2, F.Cu at (107.2, 116.7)
- added H31: MountingHole, MountingHole:MountingHole_2.2mm_M2, F.Cu at (126.2, 116.7)
- added H32: MountingHole, MountingHole:MountingHole_2.2mm_M2, F.Cu at (59.5, 126.2)
- added H33: MountingHole, MountingHole:MountingHole_2.2mm_M2, F.Cu at (78.6, 126.2)
- added H34: MountingHole, MountingHole:MountingHole_2.2mm_M2, F.Cu at (97.6, 126.2)
- added H35: MountingHole, MountingHole:MountingHole_2.2mm_M2, F.Cu at (116.7, 126.2)
- added H36: MountingHole, MountingHole:MountingHole_2.2mm_M2, F.Cu at (135.7, 126.2)
- added H37: MountingHole, MountingHole:MountingHole_2.2mm_M2, F.Cu at (69.0, 135.7)
- added H38: MountingHole, MountingHole:MountingHole_2.2mm_M2, F.Cu at (88.1, 135.7)
- added H39: MountingHole, MountingHole:MountingHole_2.2mm_M2, F.Cu at (107.2, 135.7)
- added H4: MountingHole, MountingHole:MountingHole_2.2mm_M2, F.Cu at (126.2, 59.5)
- added H40: MountingHole, MountingHole:MountingHole_2.2mm_M2, F.Cu at (126.2, 135.7)
- added H5: MountingHole, MountingHole:MountingHole_2.2mm_M2, F.Cu at (59.5, 69.0)
- added H6: MountingHole, MountingHole:MountingHole_2.2mm_M2, F.Cu at (78.6, 69.0)
- added H7: MountingHole, MountingHole:MountingHole_2.2mm_M2, F.Cu at (97.6, 69.0)
- added H8: MountingHole, MountingHole:MountingHole_2.2mm_M2, F.Cu at (116.7, 69.0)
- added H9: MountingHole, MountingHole:MountingHole_2.2mm_M2, F.Cu at (135.7, 69.0)
- added J1: Conn_01x04, footprints:conn_4, F.Cu at (73.2, 60.2)
- added J10: Conn_01x02, footprints:conn_2, F.Cu at (92.3, 63.4)
- added J100: Conn_01x04, footprints:conn_4, F.Cu at (141.1, 136.4)
- added J11: Conn_01x01, footprints:conn_1, F.Cu at (98.6, 64.9)
- added J12: Conn_01x04, footprints:conn_4, F.Cu at (103.0, 60.2)
- added J13: Conn_01x04, footprints:conn_4, F.Cu at (111.3, 60.2)
- added J14: Conn_01x02, footprints:conn_2, F.Cu at (111.3, 63.4)
- added J15: Conn_01x01, footprints:conn_1, F.Cu at (117.7, 64.9)
- added J16: Conn_01x04, footprints:conn_4, F.Cu at (122.0, 60.2)
- added J17: Conn_01x04, footprints:conn_4, F.Cu at (130.4, 60.2)
- added J18: Conn_01x02, footprints:conn_2, F.Cu at (130.4, 63.4)
- added J19: Conn_01x01, footprints:conn_1, F.Cu at (136.7, 64.9)
- added J2: Conn_01x02, footprints:conn_2, F.Cu at (73.2, 63.4)
- added J20: Conn_01x04, footprints:conn_4, F.Cu at (141.1, 60.2)
- added J21: Conn_01x04, footprints:conn_4, F.Cu at (141.1, 79.2)
- added J22: Conn_01x02, footprints:conn_2, F.Cu at (130.4, 82.5)
- added J23: Conn_01x01, footprints:conn_1, F.Cu at (136.7, 83.9)
- added J24: Conn_01x04, footprints:conn_4, F.Cu at (130.4, 79.2)
- added J25: Conn_01x04, footprints:conn_4, F.Cu at (122.0, 79.2)
- added J26: Conn_01x02, footprints:conn_2, F.Cu at (111.3, 82.5)
- added J27: Conn_01x01, footprints:conn_1, F.Cu at (117.7, 83.9)
- added J28: Conn_01x04, footprints:conn_4, F.Cu at (111.3, 79.2)
- added J29: Conn_01x04, footprints:conn_4, F.Cu at (103.0, 79.2)
- added J3: Conn_01x01, footprints:conn_1, F.Cu at (79.6, 64.9)
- added J30: Conn_01x02, footprints:conn_2, F.Cu at (92.3, 82.5)
- added J31: Conn_01x01, footprints:conn_1, F.Cu at (98.6, 83.9)
- added J32: Conn_01x04, footprints:conn_4, F.Cu at (92.3, 79.2)
- added J33: Conn_01x04, footprints:conn_4, F.Cu at (83.9, 79.2)
- added J34: Conn_01x02, footprints:conn_2, F.Cu at (73.2, 82.5)
- added J35: Conn_01x01, footprints:conn_1, F.Cu at (79.6, 83.9)
- added J36: Conn_01x04, footprints:conn_4, F.Cu at (73.2, 79.2)
- added J37: Conn_01x04, footprints:conn_4, F.Cu at (64.9, 79.2)
- added J38: Conn_01x02, footprints:conn_2, F.Cu at (54.2, 82.5)
- added J39: Conn_01x01, footprints:conn_1, F.Cu at (60.5, 83.9)
- added J4: Conn_01x04, footprints:conn_4, F.Cu at (83.9, 60.2)
- added J40: Conn_01x04, footprints:conn_4, F.Cu at (54.2, 79.2)
- added J41: Conn_01x04, footprints:conn_4, F.Cu at (54.2, 98.3)
- added J42: Conn_01x02, footprints:conn_2, F.Cu at (54.2, 101.5)
- added J43: Conn_01x01, footprints:conn_1, F.Cu at (60.5, 103.0)
- added J44: Conn_01x04, footprints:conn_4, F.Cu at (64.9, 98.3)
- added J45: Conn_01x04, footprints:conn_4, F.Cu at (73.2, 98.3)
- added J46: Conn_01x02, footprints:conn_2, F.Cu at (73.2, 101.5)
- added J47: Conn_01x01, footprints:conn_1, F.Cu at (79.6, 103.0)
- added J48: Conn_01x04, footprints:conn_4, F.Cu at (83.9, 98.3)
- added J49: Conn_01x04, footprints:conn_4, F.Cu at (92.3, 98.3)
- added J5: Conn_01x04, footprints:conn_4, F.Cu at (54.2, 60.2)
- added J50: Conn_01x02, footprints:conn_2, F.Cu at (92.3, 101.5)
- added J51: Conn_01x01, footprints:conn_1, F.Cu at (98.6, 103.0)
- added J52: Conn_01x04, footprints:conn_4, F.Cu at (103.0, 98.3)
- added J53: Conn_01x04, footprints:conn_4, F.Cu at (111.3, 98.3)
- added J54: Conn_01x02, footprints:conn_2, F.Cu at (111.3, 101.5)
- added J55: Conn_01x01, footprints:conn_1, F.Cu at (117.7, 103.0)
- added J56: Conn_01x04, footprints:conn_4, F.Cu at (122.0, 98.3)
- added J57: Conn_01x04, footprints:conn_4, F.Cu at (130.4, 98.3)
- added J58: Conn_01x02, footprints:conn_2, F.Cu at (130.4, 101.5)
- added J59: Conn_01x01, footprints:conn_1, F.Cu at (136.7, 103.0)
- added J6: Conn_01x02, footprints:conn_2, F.Cu at (54.2, 63.4)
- added J60: Conn_01x04, footprints:conn_4, F.Cu at (141.1, 98.3)
- added J61: Conn_01x04, footprints:conn_4, F.Cu at (141.1, 117.3)
- added J62: Conn_01x02, footprints:conn_2, F.Cu at (130.4, 120.6)
- added J63: Conn_01x01, footprints:conn_1, F.Cu at (136.7, 122.0)
- added J64: Conn_01x04, footprints:conn_4, F.Cu at (130.4, 117.3)
- added J65: Conn_01x04, footprints:conn_4, F.Cu at (122.0, 117.3)
- added J66: Conn_01x02, footprints:conn_2, B.Cu at (111.3, 120.6)
- added J67: Conn_01x01, footprints:conn_1, B.Cu at (117.7, 122.0)
- added J68: Conn_01x04, footprints:conn_4, F.Cu at (111.3, 117.3)
- added J69: Conn_01x04, footprints:conn_4, F.Cu at (103.0, 117.3)
- added J7: Conn_01x01, footprints:conn_1, F.Cu at (60.5, 64.9)
- added J70: Conn_01x02, footprints:conn_2, F.Cu at (92.3, 120.6)
- added J71: Conn_01x01, footprints:conn_1, F.Cu at (98.6, 122.0)
- added J72: Conn_01x04, footprints:conn_4, F.Cu at (92.3, 117.3)
- added J73: Conn_01x04, footprints:conn_4, F.Cu at (83.9, 117.3)
- added J74: Conn_01x02, footprints:conn_2, F.Cu at (73.2, 120.6)
- added J75: Conn_01x01, footprints:conn_1, F.Cu at (79.6, 122.0)
- added J76: Conn_01x04, footprints:conn_4, F.Cu at (73.2, 117.3)
- added J77: Conn_01x04, footprints:conn_4, F.Cu at (64.9, 117.3)
- added J78: Conn_01x02, footprints:conn_2, F.Cu at (54.2, 120.6)
- added J79: Conn_01x01, footprints:conn_1, F.Cu at (60.5, 122.0)
- added J8: Conn_01x04, footprints:conn_4, F.Cu at (64.9, 60.2)
- added J80: Conn_01x04, footprints:conn_4, F.Cu at (54.2, 117.3)
- added J81: Conn_01x04, footprints:conn_4, F.Cu at (54.2, 136.4)
- added J82: Conn_01x02, footprints:conn_2, F.Cu at (54.2, 139.6)
- added J83: Conn_01x01, footprints:conn_1, F.Cu at (60.5, 141.1)
- added J84: Conn_01x04, footprints:conn_4, F.Cu at (64.9, 136.4)
- added J85: Conn_01x04, footprints:conn_4, F.Cu at (73.2, 136.4)
- added J86: Conn_01x02, footprints:conn_2, F.Cu at (73.2, 139.6)
- added J87: Conn_01x01, footprints:conn_1, F.Cu at (79.6, 141.1)
- added J88: Conn_01x04, footprints:conn_4, F.Cu at (83.9, 136.4)
- added J89: Conn_01x04, footprints:conn_4, F.Cu at (92.3, 136.4)
- added J9: Conn_01x04, footprints:conn_4, F.Cu at (92.3, 60.2)
- added J90: Conn_01x02, footprints:conn_2, F.Cu at (92.3, 139.6)
- added J91: Conn_01x01, footprints:conn_1, F.Cu at (98.6, 141.1)
- added J92: Conn_01x04, footprints:conn_4, F.Cu at (103.0, 136.4)
- added J93: Conn_01x04, footprints:conn_4, F.Cu at (111.3, 136.4)
- added J94: Conn_01x02, footprints:conn_2, F.Cu at (111.3, 139.6)
- added J95: Conn_01x01, footprints:conn_1, F.Cu at (117.7, 141.1)
- added J96: Conn_01x04, footprints:conn_4, F.Cu at (122.0, 136.4)
- added J97: Conn_01x04, footprints:conn_4, F.Cu at (130.4, 136.4)
- added J98: Conn_01x02, footprints:conn_2, F.Cu at (130.4, 139.6)
- added J99: Conn_01x01, footprints:conn_1, F.Cu at (136.7, 141.1)
- added N1: VoidSwitch Footprint, footprints:VoidSwitch, F.Cu at (116.7, 59.5)
- added N10: VoidSwitch Footprint, footprints:VoidSwitch, F.Cu at (97.6, 78.6)
- added N11: VoidSwitch Footprint, footprints:VoidSwitch, F.Cu at (135.7, 97.6)
- added N12: VoidSwitch Footprint, footprints:VoidSwitch, F.Cu at (97.6, 97.6)
- added N13: VoidSwitch Footprint, footprints:VoidSwitch, F.Cu at (78.6, 97.6)
- added N14: VoidSwitch Footprint, footprints:VoidSwitch, F.Cu at (59.5, 97.6)
- added N15: VoidSwitch Footprint, footprints:VoidSwitch, F.Cu at (116.8, 97.6)
- added N16: VoidSwitch Footprint, footprints:VoidSwitch, F.Cu at (135.7, 116.7)
- added N17: VoidSwitch Footprint, footprints:VoidSwitch, F.Cu at (97.6, 116.7)
- added N18: VoidSwitch Footprint, footprints:VoidSwitch, F.Cu at (116.7, 116.7)
- added N19: VoidSwitch Footprint, footprints:VoidSwitch, F.Cu at (59.5, 116.7)
- added N2: VoidSwitch Footprint, footprints:VoidSwitch, F.Cu at (135.7, 59.5)
- added N20: VoidSwitch Footprint, footprints:VoidSwitch, F.Cu at (78.6, 116.7)
- added N21: VoidSwitch Footprint, footprints:VoidSwitch, F.Cu at (59.5, 135.7)
- added N22: VoidSwitch Footprint, footprints:VoidSwitch, F.Cu at (97.6, 135.7)
- added N23: VoidSwitch Footprint, footprints:VoidSwitch, F.Cu at (116.7, 135.7)
- added N24: VoidSwitch Footprint, footprints:VoidSwitch, F.Cu at (135.7, 135.7)
- added N25: VoidSwitch Footprint, footprints:VoidSwitch, F.Cu at (78.6, 135.7)
- added N3: VoidSwitch Footprint, footprints:VoidSwitch, F.Cu at (59.5, 59.5)
- added N4: VoidSwitch Footprint, footprints:VoidSwitch, F.Cu at (78.6, 59.5)
- added N5: VoidSwitch Footprint, footprints:VoidSwitch, F.Cu at (97.6, 59.5)
- added N6: VoidSwitch Footprint, footprints:VoidSwitch, F.Cu at (116.7, 78.6)
- added N7: VoidSwitch Footprint, footprints:VoidSwitch, F.Cu at (78.6, 78.6)
- added N8: VoidSwitch Footprint, footprints:VoidSwitch, F.Cu at (135.7, 78.6)
- added N9: VoidSwitch Footprint, footprints:VoidSwitch, F.Cu at (59.5, 78.6)
- added REF**: arrows, footprints:arrows, F.Cu at (88.1, 116.7)
- added REF**: arrows, footprints:arrows, F.Cu at (59.5, 126.2)
- added REF**: arrows, footprints:arrows, F.Cu at (88.1, 97.6)
- added REF**: arrows, footprints:arrows, F.Cu at (135.7, 69.0)
- added REF**: arrows, footprints:arrows, F.Cu at (126.2, 116.7)
- added REF**: arrows, footprints:arrows, F.Cu at (69.0, 135.7)
- added REF**: arrows, footprints:arrows, F.Cu at (126.2, 59.5)
- added REF**: arrows, footprints:arrows, F.Cu at (107.2, 97.6)
- added REF**: arrows, footprints:arrows, F.Cu at (88.1, 78.6)
- added REF**: arrows, footprints:arrows, F.Cu at (107.2, 116.7)
- added REF**: arrows, footprints:arrows, F.Cu at (126.2, 135.7)
- added REF**: arrows, footprints:arrows, F.Cu at (135.7, 107.2)
- added REF**: arrows, footprints:arrows, F.Cu at (69.0, 59.5)
- added REF**: arrows, footprints:arrows, F.Cu at (126.2, 97.6)
- added REF**: arrows, footprints:arrows, F.Cu at (88.1, 59.5)
- added REF**: arrows, footprints:arrows, F.Cu at (69.0, 78.6)
- added REF**: arrows, footprints:arrows, F.Cu at (107.2, 135.7)
- added REF**: arrows, footprints:arrows, F.Cu at (69.0, 116.7)
- added REF**: arrows, footprints:arrows, F.Cu at (107.2, 78.6)
- added REF**: arrows, footprints:arrows, F.Cu at (69.0, 97.6)
- added REF**: arrows, footprints:arrows, F.Cu at (126.2, 78.6)
- added REF**: arrows, footprints:arrows, F.Cu at (59.5, 88.1)
- added REF**: arrows, footprints:arrows, F.Cu at (107.2, 59.5)
- added REF**: arrows, footprints:arrows, F.Cu at (88.1, 135.7)
- added U1: Hall Sensor, Package_TO_SOT_SMD:SOT-23, F.Cu at (119.9, 62.8)
- added U10: SK9822, LED_SMD:LED_RGB_5050-6, F.Cu at (97.6, 59.5)
- added U11: Hall Sensor, Package_TO_SOT_SMD:SOT-23, F.Cu at (119.9, 81.8)
- added U12: SK9822, LED_SMD:LED_RGB_5050-6, F.Cu at (116.7, 78.6)
- added U13: Hall Sensor, Package_TO_SOT_SMD:SOT-23, F.Cu at (81.8, 81.8)
- added U14: SK9822, LED_SMD:LED_RGB_5050-6, F.Cu at (78.6, 78.6)
- added U15: Hall Sensor, Package_TO_SOT_SMD:SOT-23, F.Cu at (139.0, 81.8)
- added U16: SK9822, LED_SMD:LED_RGB_5050-6, F.Cu at (135.7, 78.6)
- added U17: Hall Sensor, Package_TO_SOT_SMD:SOT-23, F.Cu at (62.8, 81.8)
- added U18: SK9822, LED_SMD:LED_RGB_5050-6, F.Cu at (59.5, 78.6)
- added U19: Hall Sensor, Package_TO_SOT_SMD:SOT-23, F.Cu at (100.9, 81.8)
- added U2: SK9822, LED_SMD:LED_RGB_5050-6, F.Cu at (116.7, 59.5)
- added U20: SK9822, LED_SMD:LED_RGB_5050-6, F.Cu at (97.6, 78.6)
- added U21: Hall Sensor, Package_TO_SOT_SMD:SOT-23, F.Cu at (139.0, 100.9)
- added U22: SK9822, LED_SMD:LED_RGB_5050-6, F.Cu at (135.7, 97.6)
- added U23: Hall Sensor, Package_TO_SOT_SMD:SOT-23, F.Cu at (100.9, 100.9)
- added U24: SK9822, LED_SMD:LED_RGB_5050-6, F.Cu at (97.6, 97.6)
- added U25: Hall Sensor, Package_TO_SOT_SMD:SOT-23, F.Cu at (81.8, 100.9)
- added U26: SK9822, LED_SMD:LED_RGB_5050-6, F.Cu at (78.6, 97.6)
- added U27: Hall Sensor, Package_TO_SOT_SMD:SOT-23, F.Cu at (62.8, 100.9)
- added U28: SK9822, LED_SMD:LED_RGB_5050-6, F.Cu at (59.5, 97.6)
- added U29: Hall Sensor, Package_TO_SOT_SMD:SOT-23, F.Cu at (119.9, 100.9)
- added U3: Hall Sensor, Package_TO_SOT_SMD:SOT-23, F.Cu at (139.0, 62.8)
- added U30: SK9822, LED_SMD:LED_RGB_5050-6, F.Cu at (116.7, 97.6)
- added U31: Hall Sensor, Package_TO_SOT_SMD:SOT-23, F.Cu at (139.0, 119.9)
- added U32: SK9822, LED_SMD:LED_RGB_5050-6, F.Cu at (135.7, 116.7)
- added U33: Hall Sensor, Package_TO_SOT_SMD:SOT-23, F.Cu at (100.9, 119.9)
- added U34: SK9822, LED_SMD:LED_RGB_5050-6, F.Cu at (97.6, 116.7)
- added U35: Hall Sensor, Package_TO_SOT_SMD:SOT-23, F.Cu at (119.9, 119.9)
- added U36: SK9822, LED_SMD:LED_RGB_5050-6, F.Cu at (116.7, 116.7)
- added U37: Hall Sensor, Package_TO_SOT_SMD:SOT-23, F.Cu at (62.8, 119.9)
- added U38: SK9822, LED_SMD:LED_RGB_5050-6, F.Cu at (59.5, 116.7)
- added U39: Hall Sensor, Package_TO_SOT_SMD:SOT-23, F.Cu at (81.8, 119.9)
- added U4: SK9822, LED_SMD:LED_RGB_5050-6, F.Cu at (135.7, 59.5)
- added U40: SK9822, LED_SMD:LED_RGB_5050-6, F.Cu at (78.6, 116.7)
- added U41: Hall Sensor, Package_TO_SOT_SMD:SOT-23, F.Cu at (62.8, 139.0)
- added U42: SK9822, LED_SMD:LED_RGB_5050-6, F.Cu at (59.5, 135.7)
- added U43: Hall Sensor, Package_TO_SOT_SMD:SOT-23, F.Cu at (100.9, 139.0)
- added U44: SK9822, LED_SMD:LED_RGB_5050-6, F.Cu at (97.6, 135.7)
- added U45: Hall Sensor, Package_TO_SOT_SMD:SOT-23, F.Cu at (119.9, 139.0)
- added U46: SK9822, LED_SMD:LED_RGB_5050-6, F.Cu at (116.7, 135.7)
- added U47: Hall Sensor, Package_TO_SOT_SMD:SOT-23, F.Cu at (139.0, 139.0)
- added U48: SK9822, LED_SMD:LED_RGB_5050-6, F.Cu at (135.7, 135.7)
- added U49: Hall Sensor, Package_TO_SOT_SMD:SOT-23, F.Cu at (81.8, 139.0)
- added U5: Hall Sensor, Package_TO_SOT_SMD:SOT-23, F.Cu at (62.8, 62.8)
- added U50: SK9822, LED_SMD:LED_RGB_5050-6, F.Cu at (78.6, 135.7)
- added U6: SK9822, LED_SMD:LED_RGB_5050-6, F.Cu at (59.5, 59.5)
- added U7: Hall Sensor, Package_TO_SOT_SMD:SOT-23, F.Cu at (81.8, 62.8)
- added U8: SK9822, LED_SMD:LED_RGB_5050-6, F.Cu at (78.6, 59.5)
- added U9: Hall Sensor, Package_TO_SOT_SMD:SOT-23, F.Cu at (100.9, 62.8)
- added locked: MountingHole, MountingHole:MountingHole_2.2mm_M2, F.Cu at (107.2, 78.6)
Routing:
- net V_LED: track 0.00 -> 1786.3 mm
- net GND_HALL: track 0.00 -> 1573.8 mm, vias 0 -> 26
- net V_HALL: track 0.00 -> 689.6 mm
- net GND_LED: track 0.00 -> 629.5 mm, vias 0 -> 128
- net /Module10/SDI_LED: track 0.00 -> 58.7 mm, vias 0 -> 3
- net /Module18/SDO_LED: track 0.00 -> 58.7 mm, vias 0 -> 3
- net /Module4/SDO_LED: track 0.00 -> 57.4 mm, vias 0 -> 5
- net /Module13/SDO_LED: track 0.00 -> 57.1 mm, vias 0 -> 5
- net /Module13/CKO_LED: track 0.00 -> 56.0 mm, vias 0 -> 2
- net /Module4/CKO_LED: track 0.00 -> 56.0 mm, vias 0 -> 2
- net /Module10/CKI_LED: track 0.00 -> 49.8 mm, vias 0 -> 3
- net /Module18/CKO_LED: track 0.00 -> 49.8 mm, vias 0 -> 3
- net /Module17/SDO_LED: track 0.00 -> 44.5 mm, vias 0 -> 6
- net /Module15/SDO_LED: track 0.00 -> 44.5 mm, vias 0 -> 6
- net /Module7/SDO_LED: track 0.00 -> 44.5 mm, vias 0 -> 6
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- added copper zone on B.Cu, net GND_HALL
- added copper zone on B.Cu, net GND_LED
- added copper zone on F.Cu, net GND_LED
Other:
- board size 225.7 x 100.8 mm -> 95.2 x 95.2 mm
- board text added: "CKI"
- board text added: "CKO"
- board text added: "GLED"
- board text added: "GNDH"
- board text added: "GNDL"
- board text added: "HALL"
- board text added: "SDI"
- board text added: "SDO"
- board text added: "VCCH"
- board text added: "VCCL"
- board text added: "VLED"
- board text added: "https://0jb.de/akhm"
- board text removed: "{{GITHASH}}"
